Commit message: 微调了URDF的关节限制，修正了关节初始角度

File: src/dog/urdf/dog.urdf (robot description, URDF)
Before this commit: robot dog, 13 links, 12 joints
Joints:
- joint lb_joint1: axis 0 0 0 -> 0 0 1; limit lower=0 upper=0 effort=0 velocity=0 -> lower=-1.851 upper=0.425 effort=0 velocity=0
- joint lb_joint2: axis 0 0 0 -> 0 0 1; limit lower=0 upper=0 effort=0 velocity=0 -> lower=-3.14159265 upper=3.14159265 effort=0 velocity=0; origin xyz=0 -0.0046 0.06233 rpy=1.5708 -0.28365 0 -> xyz=0 -0.0046 0.06233 rpy=1.5708 0 0
- joint lb_joint3: axis 0 0 0 -> 0 0 1; limit lower=0 upper=0 effort=0 velocity=0 -> lower=-2.836 upper=-0.628 effort=0 velocity=0; origin xyz=0.2299 -0.0066352 0.0711 rpy=0 0 -0.76946 -> xyz=0.2299 -0.0066352 0.0711 rpy=0 0 0
- joint lf_joint1: axis 0 0 -1 -> 0 0 1; limit lower=0 upper=0 effort=0 velocity=0 -> lower=-0.425 upper=1.851 effort=0 velocity=0
- joint lf_joint2: limit lower=0 upper=0 effort=0 velocity=0 -> lower=-3.14159265 upper=3.14159265 effort=0 velocity=0; origin xyz=0 0.0046 0.06233 rpy=-1.5708 0.715 0 -> xyz=0 0.0046 0.06233 rpy=-1.5708 0 0
- joint lf_joint3: limit lower=0 upper=0 effort=0 velocity=0 -> lower=0.628 upper=2.836 effort=0 velocity=0; origin xyz=0.22851 -0.026109 0.0711 rpy=0 0 -1.4148 -> xyz=0.22851 -0.026109 0.0711 rpy=0 0 0
- joint rb_joint1: axis 0 0 0 -> 0 0 1; limit lower=0 upper=0 effort=0 velocity=0 -> lower=-0.425 upper=1.851 effort=0 velocity=0
- joint rb_joint2: axis 0 0 0 -> 0 0 1; limit lower=0 upper=0 effort=0 velocity=0 -> lower=-3.14159265 upper=3.14159265 effort=0 velocity=0; origin xyz=0 0.0046 0.06233 rpy=-1.5708 -0.78295 0 -> xyz=0 0.0046 0.06233 rpy=-1.5708 0 0
- joint rb_joint3: axis 0 0 0 -> 0 0 1; limit lower=0 upper=0 effort=0 velocity=0 -> lower=0.628 upper=2.836 effort=0 velocity=0; origin xyz=0.22851 0.026109 0.0711 rpy=0 0 1.5163 -> xyz=0.22851 0.026109 0.0711 rpy=0 0 0
- joint rf_joint1: axis 0 0 0 -> 0 0 1; limit lower=0 upper=0 effort=0 velocity=0 -> lower=-1.851 upper=0.425 effort=0 velocity=0
- joint rf_joint2: axis 0 0 0 -> 0 0 1; limit lower=0 upper=0 effort=0 velocity=0 -> lower=-3.14159265 upper=3.14159265 effort=0 velocity=0; origin xyz=-0.00024992 -0.0044 0.06233 rpy=1.5708 0.71388 0 -> xyz=-0.00024992 -0.0044 0.06233 rpy=1.5708 0 0
- joint rf_joint3: axis 0 0 0 -> 0 0 1; limit lower=0 upper=0 effort=0 velocity=0 -> lower=0.628 upper=2.836 effort=0 velocity=0; origin xyz=0.22851 0.026109 0.0711 rpy=0 0 1.1184 -> xyz=0.22851 0.026109 0.0711 rpy=0 0 0

Commit message: 重新导出了mesh文件和URDF文件，修正了URDF文件

File: src/dog/urdf/dog.urdf (robot description, URDF)
Before this commit: robot dog, 13 links, 12 joints
Links:
- added link lb_link4, mass 0.0869238618825574; collision mesh filename=package://dog/meshes/lb_link4.STL; visual mesh filename=package://dog/meshes/lb_link4.STL
- added link lf_link4, mass 0.0869238618825573; collision mesh filename=package://dog/meshes/lf_link4.STL; visual mesh filename=package://dog/meshes/lf_link4.STL
- added link rb_link4, mass 0.0825104582750147; collision mesh filename=package://dog/meshes/rb_link4.STL; visual mesh filename=package://dog/meshes/rb_link4.STL
- added link rf_link4, mass 0.0825104582750148; collision mesh filename=package://dog/meshes/rf_link4.STL; visual mesh filename=package://dog/meshes/rf_link4.STL
- link body_link: mass 1.2602016062932 -> 1.26020160629337
- link lb_link1: mass 0.345687127151886 -> 0.445687127151886
- link lb_link2: mass 0.684092508880398 -> 0.684092508880399
- link lb_link3: mass 0.591391038477536 -> 0.501282068000102
- link lf_link1: mass 0.334681727936514 -> 0.449515096090149
- link lf_link3: mass 0.580292054459404 -> 0.496989020503303
- link rb_link1: mass 0.308609260085749 -> 0.408609260085749
- link rb_link2: mass 0.643709660125423 -> 0.669259133619637
- link rb_link3: mass 0.586977638584799 -> 0.501282071766371
- link rf_link1: mass 0.345687130115019 -> 0.44568713011502
- link rf_link2: mass 0.660568167276523 -> 0.619089741901032
- link rf_link3: mass 0.586977638952076 -> 0.501282072155041
Joints:
- added joint lb_joint4: type fixed, parent lb_link3, child lb_link4, origin xyz=0.24 0 0.0238 rpy=0 0 0, axis 0 0 0
- added joint lf_link4: type fixed, parent lf_link3, child lf_link4, origin xyz=0.24 0 0.0238 rpy=0 0 0, axis 0 0 0
- added joint rb_joint4: type fixed, parent rb_link3, child rb_link4, origin xyz=0.24 0 0.0238 rpy=0 0 0, axis 0 0 0
- added joint rf_joint4: type fixed, parent rf_link3, child rf_link4, origin xyz=0.24 0 0.0238 rpy=0 0 0, axis 0 0 0
- joint lb_joint1: limit lower=-1.851 upper=0.425 effort=0 velocity=0 -> lower=-1.953 upper=0.4 effort=0 velocity=0
- joint lb_joint2: limit lower=-3.14159265 upper=3.14159265 effort=0 velocity=0 -> lower=-3.14159 upper=3.14159 effort=0 velocity=0
- joint lb_joint3: limit lower=-2.836 upper=-0.628 effort=0 velocity=0 -> lower=-1.240 upper=1.274 effort=0 velocity=0; origin xyz=0.2299 -0.0066352 0.0711 rpy=0 0 0 -> xyz=0.2299 -0.0066352 0.0711 rpy=0 0 -1.5708
- joint lf_joint1: limit lower=-0.425 upper=1.851 effort=0 velocity=0 -> lower=-0.4 upper=1.953 effort=0 velocity=0
- joint lf_joint2: limit lower=-3.14159265 upper=3.14159265 effort=0 velocity=0 -> lower=-3.14159 upper=3.14159 effort=0 velocity=0
- joint lf_joint3: axis 0 0 -1 -> 0 0 1; limit lower=0.628 upper=2.836 effort=0 velocity=0 -> lower=-1.274 upper=1.240 effort=0 velocity=0; origin xyz=0.22851 -0.026109 0.0711 rpy=0 0 0 -> xyz=0.22851 -0.026109 0.0711 rpy=0 0 -1.5708
- joint rb_joint1: limit lower=-0.425 upper=1.851 effort=0 velocity=0 -> lower=-0.4 upper=1.953 effort=0 velocity=0; origin xyz=-0.1916 -0.09 0.052 rpy=1.5708 1.5334 -1.5708 -> xyz=-0.1916 -0.09 0.052 rpy=1.5708 1.5708 -1.5708
- joint rb_joint2: limit lower=-3.14159265 upper=3.14159265 effort=0 velocity=0 -> lower=-3.14159 upper=3.14159 effort=0 velocity=0
- joint rb_joint3: limit lower=0.628 upper=2.836 effort=0 velocity=0 -> lower=-1.274 upper=1.240 effort=0 velocity=0; origin xyz=0.22851 0.026109 0.0711 rpy=0 0 0 -> xyz=0.22851 0.026109 0.0711 rpy=0 0 1.5708
- joint rf_joint1: limit lower=-1.851 upper=0.425 effort=0 velocity=0 -> lower=-1.953 upper=0.4 effort=0 velocity=0
- joint rf_joint2: limit lower=-3.14159265 upper=3.14159265 effort=0 velocity=0 -> lower=-3.14159 upper=3.14159 effort=0 velocity=0; origin xyz=-0.00024992 -0.0044 0.06233 rpy=1.5708 0 0 -> xyz=-0.00024992 -0.0044 0.06233 rpy=1.5708 0.0 0
- joint rf_joint3: limit lower=0.628 upper=2.836 effort=0 velocity=0 -> lower=-1.240 upper=1.274 effort=0 velocity=0; origin xyz=0.22851 0.026109 0.0711 rpy=0 0 0 -> xyz=0.22851 0.026109 0.0711 rpy=0 0 1.5708

Commit message: 1

File: src/dog/urdf/dog.urdf (robot description, URDF)
Before this commit: robot dog, 17 links, 16 joints
Joints:
- removed joint lf_link4
- added joint lf_joint4: type fixed, parent lf_link3, child lf_link4, origin xyz=0.24 0 0.0238 rpy=0 0 0, axis 0 0 0

Commit message: 完成了基本的运行Gazebo仿真，遇到了仿真速度特别慢的问题

File: src/dog/urdf/dog.urdf (robot description, URDF)
Before this commit: robot dog, 17 links, 16 joints
Joints:
- joint lb_joint1: limit lower=-1.953 upper=0.4 effort=0 velocity=0 -> lower=-1.953 upper=0.4 effort=20 velocity=20
- joint lb_joint2: limit lower=-3.14159 upper=3.14159 effort=0 velocity=0 -> lower=-3.14159 upper=3.14159 effort=20 velocity=20
- joint lb_joint3: limit lower=-1.240 upper=1.274 effort=0 velocity=0 -> lower=-1.240 upper=1.274 effort=20 velocity=20
- joint lf_joint1: limit lower=-0.4 upper=1.953 effort=0 velocity=0 -> lower=-0.4 upper=1.953 effort=20 velocity=20
- joint lf_joint2: limit lower=-3.14159 upper=3.14159 effort=0 velocity=0 -> lower=-3.14159 upper=3.14159 effort=20 velocity=20
- joint lf_joint3: limit lower=-1.274 upper=1.240 effort=0 velocity=0 -> lower=-1.274 upper=1.240 effort=20 velocity=20
- joint rb_joint1: limit lower=-0.4 upper=1.953 effort=0 velocity=0 -> lower=-0.4 upper=1.953 effort=20 velocity=20
- joint rb_joint2: limit lower=-3.14159 upper=3.14159 effort=0 velocity=0 -> lower=-3.14159 upper=3.14159 effort=20 velocity=20
- joint rb_joint3: limit lower=-1.274 upper=1.240 effort=0 velocity=0 -> lower=-1.274 upper=1.240 effort=20 velocity=20
- joint rf_joint1: limit lower=-1.953 upper=0.4 effort=0 velocity=0 -> lower=-1.953 upper=0.4 effort=20 velocity=20
- joint rf_joint2: limit lower=-3.14159 upper=3.14159 effort=0 velocity=0 -> lower=-3.14159 upper=3.14159 effort=20 velocity=20
- joint rf_joint3: limit lower=-1.240 upper=1.274 effort=0 velocity=0 -> lower=-1.240 upper=1.274 effort=20 velocity=20

Commit message: 完成了完整的PID在线调参和Gazebo步态仿真

File: src/dog/urdf/dog.urdf (robot description, URDF)
Before this commit: robot dog, 17 links, 16 joints
Links:
- link lb_link4: geometry collision sphere radius=0.06; visual mesh filename=package://dog/meshes/lb_link4.STL
- link lf_link4: geometry collision sphere radius=0.06; visual mesh filename=package://dog/meshes/lf_link4.STL
- link rb_link4: geometry collision sphere radius=0.06; visual mesh filename=package://dog/meshes/rb_link4.STL
- link rf_link4: geometry collision sphere radius=0.06; visual mesh filename=package://dog/meshes/rf_link4.STL

Commit message: 使用第二代狗子的URDF模型

File: src/dog/urdf/dog.urdf (robot description, URDF)
Before this commit: robot dog, 17 links, 16 joints
Links:
- link body_link: mass 1.26020160629337 -> 3.0135
- link lb_link1: mass 0.445687127151886 -> 0.305258519686429
- link lb_link2: mass 0.684092508880399 -> 0.673603806804068
- link lb_link3: mass 0.501282068000102 -> 0.119977441819341
- link lb_link4: mass 0.0869238618825574 -> 0.0781572031669603
- link lf_link1: mass 0.449515096090149 -> 0.305258503824178
- link lf_link2: mass 0.681135261025341 -> 0.644661117972557
- link lf_link3: mass 0.496989020503303 -> 0.119977441819341
- link lf_link4: mass 0.0869238618825573 -> 0.0781571728156937
- link rb_link1: mass 0.408609260085749 -> 0.305258557068333
- link rb_link2: mass 0.669259133619637 -> 0.682338894787625
- link rb_link3: mass 0.501282071766371 -> 0.119977441819341
- link rb_link4: mass 0.0825104582750147 -> 0.0781572323930169
- link rf_link1: mass 0.44568713011502 -> 0.305258502432481
- link rf_link2: mass 0.619089741901032 -> 0.65339621713157
- link rf_link3: mass 0.501282072155041 -> 0.11997744181934
- link rf_link4: mass 0.0825104582750148 -> 0.0781571826488302
Joints:
- joint lb_joint1: axis 0 0 1 -> 0 0 -1; limit lower=-1.953 upper=0.4 effort=20 velocity=20 -> lower=-3 upper=3 effort=20 velocity=16; origin xyz=-0.1916 0.09 0.052 rpy=1.5708 1.5627 -1.5708 -> xyz=-0.1916 0.070013 0.061999 rpy=3.1416 1.5708 0
- joint lb_joint2: axis 0 0 1 -> 0 0 -1; limit lower=-3.14159 upper=3.14159 effort=20 velocity=20 -> lower=-3 upper=3 effort=20 velocity=16; origin xyz=0 -0.0046 0.06233 rpy=1.5708 0 0 -> xyz=7.0296E-05 -0.029287 0.059987 rpy=1.5708 0 0
- joint lb_joint3: axis 0 0 1 -> 0 0 -1; limit lower=-1.240 upper=1.274 effort=20 velocity=20 -> lower=-3 upper=3 effort=20 velocity=16; origin xyz=0.2299 -0.0066352 0.0711 rpy=0 0 -1.5708 -> xyz=0.23001 0 0.0935 rpy=0 0 -1.5708
- joint lb_joint4: origin xyz=0.24 0 0.0238 rpy=0 0 0 -> xyz=0.24313 0.012189 -0.023501 rpy=0 0 0
- joint lf_joint1: axis 0 0 1 -> 0 0 -1; limit lower=-0.4 upper=1.953 effort=20 velocity=20 -> lower=-3 upper=3 effort=20 velocity=16; origin xyz=0.1916 0.09 0.052 rpy=0 1.5708 0 -> xyz=0.1916 0.069987 0.061999 rpy=0 1.5708 0
- joint lf_joint2: axis 0 0 1 -> 0 0 -1; limit lower=-3.14159 upper=3.14159 effort=20 velocity=20 -> lower=-3 upper=3 effort=20 velocity=16; origin xyz=0 0.0046 0.06233 rpy=-1.5708 0 0 -> xyz=-0.000957 0.029298 0.060013 rpy=-1.5708 0 0
- joint lf_joint3: limit lower=-1.274 upper=1.240 effort=20 velocity=20 -> lower=-3 upper=3 effort=20 velocity=16; origin xyz=0.22851 -0.026109 0.0711 rpy=0 0 -1.5708 -> xyz=0.23001 0 0.0935 rpy=0 0 -1.5708
- joint lf_joint4: origin xyz=0.24 0 0.0238 rpy=0 0 0 -> xyz=0.243132280457965 0.0121889545734945 -0.0235007169194983 rpy=0 0 -3.14159265358976
- joint rb_joint1: axis 0 0 1 -> 0 0 -1; limit lower=-0.4 upper=1.953 effort=20 velocity=20 -> lower=-3 upper=3 effort=20 velocity=16; origin xyz=-0.1916 -0.09 0.052 rpy=1.5708 1.5708 -1.5708 -> xyz=-0.1916 -0.07 0.062 rpy=3.1416 1.5708 0
- joint rb_joint2: axis 0 0 1 -> 0 0 -1; limit lower=-3.14159 upper=3.14159 effort=20 velocity=20 -> lower=-3 upper=3 effort=20 velocity=16; origin xyz=0 0.0046 0.06233 rpy=-1.5708 0 0 -> xyz=-0.0022402 0.029214 0.06 rpy=-1.5708 0 0
- joint rb_joint3: axis 0 0 1 -> 0 0 -1; limit lower=-1.274 upper=1.240 effort=20 velocity=20 -> lower=-3 upper=3 effort=20 velocity=16; origin xyz=0.22851 0.026109 0.0711 rpy=0 0 1.5708 -> xyz=0.23 0 0.0935 rpy=0 0 1.5708
- joint rb_joint4: origin xyz=0.24 0 0.0238 rpy=0 0 0 -> xyz=0.24313 -0.012189 -0.023499 rpy=0 0 0
- joint rf_joint1: axis 0 0 1 -> 0 0 -1; limit lower=-1.953 upper=0.4 effort=20 velocity=20 -> lower=-3 upper=3 effort=20 velocity=16; origin xyz=0.1916 -0.09 0.052 rpy=0 1.5708 0 -> xyz=0.1916 -0.070013 0.061999 rpy=0 1.5708 0
- joint rf_joint2: limit lower=-3.14159 upper=3.14159 effort=20 velocity=20 -> lower=-3 upper=3 effort=20 velocity=16; origin xyz=-0.00024992 -0.0044 0.06233 rpy=1.5708 0.0 0 -> xyz=-0.0010387 -0.029268 0.059987 rpy=1.5708 0 0
- joint rf_joint3: axis 0 0 1 -> 0 -0.035945 -0.99935; limit lower=-1.240 upper=1.274 effort=20 velocity=20 -> lower=-3 upper=3 effort=20 velocity=16; origin xyz=0.22851 0.026109 0.0711 rpy=0 0 1.5708 -> xyz=0.22999 1.0169E-05 0.0935 rpy=0.0 0.0 1.5708
- joint rf_joint4: origin xyz=0.24 0 0.0238 rpy=0 0 0 -> xyz=0.24313 -0.013026 -0.023046 rpy=3.1056 0 0
