Commit message: 根据电机旋转方向修正URDF中关节旋转轴的正负

File: src/dog/model/dog.urdf (robot description, URDF)
Before this commit: robot dog, 17 links, 16 joints
Joints:
- joint lb_joint1: axis 0 0 -1 -> 0 0 1
- joint lb_joint2: axis 0 0 -1 -> 0 0 1
- joint lf_joint1: axis 0 0 -1 -> 0 0 1
- joint lf_joint2: axis 0 0 -1 -> 0 0 1
- joint rb_joint1: axis 0 0 -1 -> 0 0 1
- joint rb_joint2: axis 0 0 -1 -> 0 0 1
- joint rb_joint3: axis 0 0 -1 -> 0 0 1
- joint rf_joint1: axis 0 0 -1 -> 0 0 1
- joint rf_joint3: axis 0 -0.035945 -0.99935 -> 0 0 1

Commit message: 更改上电后的启动流程，在关节空间规划曲线，解决启动时因为接近奇点，进行逆解导致的不稳定问题；微调了VMC参数

File: src/dog/model/dog.urdf (robot description, URDF)
Before this commit: robot dog, 17 links, 16 joints
Links:
- link body_link: mass 3.0135 -> 4.2135
Joints:
- joint lb_joint3: axis 0 0 -1 -> 0 0 1

Commit message: 减面后的dog

File: src/dog/model/dog.urdf (robot description, URDF)
Before this commit: robot dog, 17 links, 16 joints
Links:
- link body_link: mass 3.0135 -> 3.1484; geometry collision mesh filename=package://dog/meshes/body_link.STL; visual mesh filename=package://dog/meshes/body_link.STL
- link lb_link1: mass 0.305258519686429 -> 0.305258513351168; geometry collision mesh filename=package://dog/meshes/lb_link1.STL; visual mesh filename=package://dog/meshes/lb_link1.STL
- link lb_link2: mass 0.673603806804068 -> 0.682338727402138; geometry collision mesh filename=package://dog/meshes/lb_link2.STL; visual mesh filename=package://dog/meshes/lb_link2.STL
- link lb_link3: mass 0.119977441819341 -> 0.127541149243291; geometry collision mesh filename=package://dog/meshes/lb_link3.STL; visual mesh filename=package://dog/meshes/lb_link3.STL
- link lb_link4: mass 0.0781572031669603 -> 0.433967634660258; geometry collision mesh filename=package://dog/meshes/lb_link4.STL; visual mesh filename=package://dog/meshes/lb_link4.STL
- link lf_link1: mass 0.305258503824178 -> 0.305258520873073; geometry collision mesh filename=package://dog/meshes/lf_link1.STL; visual mesh filename=package://dog/meshes/lf_link1.STL
- link lf_link2: mass 0.644661117972557 -> 0.687935232941792; geometry collision mesh filename=package://dog/meshes/lf_link2.STL; visual mesh filename=package://dog/meshes/lf_link2.STL
- link lf_link3: mass 0.119977441819341 -> 0.0715412570113013; geometry collision mesh filename=package://dog/meshes/lf_link3.STL; visual mesh filename=package://dog/meshes/lf_link3.STL
- link lf_link4: mass 0.0781571728156937 -> 0.392667576355364; geometry collision mesh filename=package://dog/meshes/lf_link4.STL; visual mesh filename=package://dog/meshes/lf_link4.STL
- link rb_link1: mass 0.305258557068333 -> 0; geometry collision mesh filename=package://dog/meshes/rb_link1.STL; visual mesh filename=package://dog/meshes/rb_link1.STL
- link rb_link2: mass 0.682338894787625 -> 0.682338713258883; geometry collision mesh filename=package://dog/meshes/rb_link2.STL; visual mesh filename=package://dog/meshes/rb_link2.STL
- link rb_link3: mass 0.119977441819341 -> 0.127541149243291; geometry collision mesh filename=package://dog/meshes/rb_link3.STL; visual mesh filename=package://dog/meshes/rb_link3.STL
- link rb_link4: mass 0.0781572323930169 -> 0.433967544275498; geometry collision mesh filename=package://dog/meshes/rb_link4.STL; visual mesh filename=package://dog/meshes/rb_link4.STL
- link rf_link1: mass 0.305258502432481 -> 0.305258520879218; geometry collision mesh filename=package://dog/meshes/rf_link1.STL; visual mesh filename=package://dog/meshes/rf_link1.STL
- link rf_link2: mass 0.65339621713157 -> 0.682338731946651; geometry collision mesh filename=package://dog/meshes/rf_link2.STL; visual mesh filename=package://dog/meshes/rf_link2.STL
- link rf_link3: mass 0.11997744181934 -> 0.127541149243291; geometry collision mesh filename=package://dog/meshes/rf_link3.STL; visual mesh filename=package://dog/meshes/rf_link3.STL
- link rf_link4: mass 0.0781571826488302 -> 0.433967655538312; geometry collision mesh filename=package://dog/meshes/rf_link4.STL; visual mesh filename=package://dog/meshes/rf_link4.STL
Joints:
- joint lb_joint1: limit lower=-3 upper=3 effort=20 velocity=16 -> lower=0 upper=0 effort=0 velocity=0; origin xyz=-0.1916 0.070013 0.061999 rpy=3.1416 1.5708 0 -> xyz=-0.191600000000032 0.0700132256966699 0.0619991926788507 rpy=3.14159265358979 1.5707963267949 0
- joint lb_joint2: limit lower=-3 upper=3 effort=20 velocity=16 -> lower=0 upper=0 effort=0 velocity=0; origin xyz=7.0296E-05 -0.029287 0.059987 rpy=1.5708 0 0 -> xyz=-0.000473865368497223 -0.0292829552273839 0.0599867742981585 rpy=-1.5707963267949 0 3.12541907549099
- joint lb_joint3: limit lower=-3 upper=3 effort=20 velocity=16 -> lower=0 upper=0 effort=0 velocity=0; origin xyz=0.23001 0 0.0935 rpy=0 0 -1.5708 -> xyz=-0.203351876537887 -0.10747338576928 0.0935000000000002 rpy=0 0 2.90766742618988
- joint lb_joint4: axis 0 0 0 -> 0 -0.0605528116672081 0.998164994877698; origin xyz=0.24313 0.012189 -0.023501 rpy=0 0 0 -> xyz=0.0844672765357189 -0.192299044270706 -0.428612988849078 rpy=3.08100277647518 0 -1.33687109939488; type fixed -> continuous
- joint lf_joint1: limit lower=-3 upper=3 effort=20 velocity=16 -> lower=0 upper=0 effort=0 velocity=0; origin xyz=0.1916 0.069987 0.061999 rpy=0 1.5708 0 -> xyz=0.191599999999968 0.0699866617468943 0.0619994644116205 rpy=0 1.5707963267949 0
- joint lf_joint2: limit lower=-3 upper=3 effort=20 velocity=16 -> lower=0 upper=0 effort=0 velocity=0; origin xyz=-0.000957 0.029298 0.060013 rpy=-1.5708 0 0 -> xyz=0 0.0293132256966799 0.060013338253096 rpy=1.5707963267949 0 3.14159265358979
- joint lf_joint3: axis 0 0 1 -> 0 0 -1; limit lower=-3 upper=3 effort=20 velocity=16 -> lower=0 upper=0 effort=0 velocity=0; origin xyz=0.23001 0 0.0935 rpy=0 0 -1.5708 -> xyz=-0.093817 -0.21001 0.0935 rpy=0 0 -1.5708
- joint lf_joint4: axis 0 0 0 -> 0 0 -1; origin xyz=0.243132280457965 0.0121889545734945 -0.0235007169194983 rpy=0 0 -3.14159265358976 -> xyz=-0.122237359979855 -0.185579634525742 0.0279999999999998 rpy=0 0 0; type fixed -> continuous
- joint rb_joint1: limit lower=-3 upper=3 effort=20 velocity=16 -> lower=0 upper=0 effort=0 velocity=0; origin xyz=-0.1916 -0.07 0.062 rpy=3.1416 1.5708 0 -> xyz=-0.191600000000032 -0.0700000000000098 0.0619999999999996 rpy=3.14159265358979 1.5707963267949 0
- joint rb_joint2: limit lower=-3 upper=3 effort=20 velocity=16 -> lower=0 upper=0 effort=0 velocity=0; origin xyz=-0.0022402 0.029214 0.06 rpy=-1.5708 0 0 -> xyz=-0.0013009697021988 0.0292711031195265 0.0600000000000002 rpy=-1.5707963267949 0 0.044416299015803
- joint rb_joint3: limit lower=-3 upper=3 effort=20 velocity=16 -> lower=0 upper=0 effort=0 velocity=0; origin xyz=0.23 0 0.0935 rpy=0 0 1.5708 -> xyz=0.19696 -0.11878 0.0935 rpy=0 0 1.32
- joint rb_joint4: axis 0 0 0 -> 0 0 -1; origin xyz=0.24313 -0.012189 -0.023499 rpy=0 0 0 -> xyz=0.225000000000112 0 0.0279999999999998 rpy=0 0 0.250835783240079; type fixed -> continuous
- joint rf_joint1: limit lower=-3 upper=3 effort=20 velocity=16 -> lower=0 upper=0 effort=0 velocity=0
- joint rf_joint2: axis 0 0 1 -> 0 0 -1; limit lower=-3 upper=3 effort=20 velocity=16 -> lower=0 upper=0 effort=0 velocity=0; origin xyz=-0.0010387 -0.029268 0.059987 rpy=1.5708 0 0 -> xyz=0 -0.0292867743011825 0.0599867742981584 rpy=1.5707963267949 -1.5707963267949 0
- joint rf_joint3: axis 0 -0.035945 -0.99935 -> 0 0 -1; limit lower=-3 upper=3 effort=20 velocity=16 -> lower=0 upper=0 effort=0 velocity=0; origin xyz=0.22999 1.0169E-05 0.0935 rpy=0.0 0.0 1.5708 -> xyz=-0.13592 -0.18553 0.0935 rpy=0 0 -0.80414
- joint rf_joint4: axis 0 0 0 -> 0 0 -1; origin xyz=0.24313 -0.013026 -0.023046 rpy=3.1056 0 0 -> xyz=0.225000000000005 0 0.0280000000000001 rpy=0 0 0.804141963898708; type fixed -> continuous

Commit message: 修改urdf，xml

File: src/dog/model/dog.urdf (robot description, URDF)
Before this commit: robot dog, 17 links, 16 joints
Links:
- link body_link: mass 4.2135 -> 3.14843748747337
- link lb_link1: mass 0.305258513351168 -> 0.30525851335117
- link lb_link2: mass 0.682338727402138 -> 0.682338727568128
- link lb_link4: mass 0.433967634660258 -> 0.432627590726503
- link lf_link1: mass 0.305258520873073 -> 0.305258520873074
- link lf_link2: mass 0.687935232941792 -> 0.687935058008792
- link lf_link3: mass 0.0715412570113013 -> 0.0715412570113012
- link lf_link4: mass 0.392667576355364 -> 0.392667576355367
- link rb_link1: mass 0 -> 0.305258497916776
- link rb_link2: mass 0.682338713258883 -> 0.682338712671128
- link rb_link4: mass 0.433967544275498 -> 0.432627455975136
- link rf_link1: mass 0.305258520879218 -> 0.305258520879219
- link rf_link2: mass 0.682338731946651 -> 0.682338731946652
- link rf_link4: mass 0.433967655538312 -> 0.43262756992202
Joints:
- joint lb_joint1: axis 0 0 1 -> 0 0 -1; origin xyz=-0.191600000000032 0.0700132256966699 0.0619991926788507 rpy=3.14159265358979 1.5707963267949 0 -> xyz=-0.1916 0.070013 0.061999 rpy=3.1416 1.5708 0
- joint lb_joint2: origin xyz=-0.000473865368497223 -0.0292829552273839 0.0599867742981585 rpy=-1.5707963267949 0 3.12541907549099 -> xyz=-0.00047387 -0.029283 0.059987 rpy=-1.5708 0 3.1254
- joint lb_joint3: axis 0 0 1 -> 0 0 -1; origin xyz=-0.203351876537887 -0.10747338576928 0.0935000000000002 rpy=0 0 2.90766742618988 -> xyz=-0.17921 -0.14417 0.0935 rpy=0 0 2.6627
- joint lb_joint4: axis 0 -0.0605528116672081 0.998164994877698 -> 0 0 -1; origin xyz=0.0844672765357189 -0.192299044270706 -0.428612988849078 rpy=3.08100277647518 0 -1.33687109939488 -> xyz=0.225 0 0.028 rpy=0 0 2.0497
- joint lf_joint1: axis 0 0 1 -> 0 0 -1; origin xyz=0.191599999999968 0.0699866617468943 0.0619994644116205 rpy=0 1.5707963267949 0 -> xyz=0.1916 0.069987 0.061999 rpy=0 1.5708 0
- joint lf_joint2: axis 0 0 1 -> 0 0 -1; origin xyz=0 0.0293132256966799 0.060013338253096 rpy=1.5707963267949 0 3.14159265358979 -> xyz=0 0.029313 0.060013 rpy=1.5708 0 3.1416
- joint lf_joint3: origin xyz=-0.093817 -0.21001 0.0935 rpy=0 0 -1.5708 -> xyz=-0.14792 -0.17613 0.0935 rpy=0 0 -1.5708
- joint lf_joint4: origin xyz=-0.122237359979855 -0.185579634525742 0.0279999999999998 rpy=0 0 0 -> xyz=-0.17165 -0.14547 0.028 rpy=0 0 0
- joint rb_joint1: axis 0 0 1 -> 0 0 -1; origin xyz=-0.191600000000032 -0.0700000000000098 0.0619999999999996 rpy=3.14159265358979 1.5707963267949 0 -> xyz=-0.1916 -0.07 0.062 rpy=3.1416 1.5708 0
- joint rb_joint2: axis 0 0 1 -> 0 0 -1; origin xyz=-0.0013009697021988 0.0292711031195265 0.0600000000000002 rpy=-1.5707963267949 0 0.044416299015803 -> xyz=-0.001301 0.029271 0.06 rpy=-1.5708 0 0.044416
- joint rb_joint3: axis 0 0 1 -> 0 0 -1; origin xyz=0.19696 -0.11878 0.0935 rpy=0 0 1.32 -> xyz=0.19386 -0.12377 0.0935 rpy=0 0 0.53404
- joint rb_joint4: origin xyz=0.225000000000112 0 0.0279999999999998 rpy=0 0 0.250835783240079 -> xyz=0.225 0 0.028 rpy=0 0 1.0368
- joint rf_joint1: axis 0 0 1 -> 0 0 -1
- joint rf_joint2: axis 0 0 1 -> 0 0 -1; origin xyz=0 -0.0292867743011825 0.0599867742981584 rpy=1.5707963267949 -1.5707963267949 0 -> xyz=0 -0.029287 0.059987 rpy=1.5708 -1.5708 0
- joint rf_joint3: axis 0 0 1 -> 0 0 -1
- joint rf_joint4: origin xyz=0.225000000000005 0 0.0280000000000001 rpy=0 0 0.804141963898708 -> xyz=0.225 0 0.028 rpy=0 0 0.80414

Commit message: 新狗模型

File: src/dog/model/dog.urdf (robot description, URDF)
Before this commit: robot dog, 17 links, 16 joints
Links:
- link body_link: mass 3.14843748747337 -> 3.1484; geometry collision mesh filename=package://dog/model/body_link.STL; visual mesh filename=package://dog/model/body_link.STL
- link lb_link1: mass 0.30525851335117 -> 0.305258513351169; geometry collision mesh filename=package://dog/model/lb_link1.STL; visual mesh filename=package://dog/model/lb_link1.STL
- link lb_link2: geometry collision mesh filename=package://dog/model/lb_link2.STL; visual mesh filename=package://dog/model/lb_link2.STL
- link lb_link3: geometry collision mesh filename=package://dog/model/lb_link3.STL; visual mesh filename=package://dog/model/lb_link3.STL
- link lb_link4: mass 0.432627590726503 -> 0.432627590726504; geometry collision mesh filename=package://dog/model/lb_link4.STL; visual mesh filename=package://dog/model/lb_link4.STL
- link lf_link1: mass 0.305258520873074 -> 0.30526; geometry collision mesh filename=package://dog/model/lf_link1.STL; visual mesh filename=package://dog/model/lf_link1.STL
- link lf_link2: mass 0.687935058008792 -> 0.687935058013005; geometry collision mesh filename=package://dog/model/lf_link2.STL; visual mesh filename=package://dog/model/lf_link2.STL
- link lf_link3: geometry collision mesh filename=package://dog/model/lf_link3.STL; visual mesh filename=package://dog/model/lf_link3.STL
- link lf_link4: geometry collision mesh filename=package://dog/model/lf_link4.STL; visual mesh filename=package://dog/model/lf_link4.STL
- link rb_link1: geometry collision mesh filename=package://dog/model/rb_link1.STL; visual mesh filename=package://dog/model/rb_link1.STL
- link rb_link2: mass 0.682338712671128 -> 0.682338712671127; geometry collision mesh filename=package://dog/model/rb_link2.STL; visual mesh filename=package://dog/model/rb_link2.STL
- link rb_link3: geometry collision mesh filename=package://dog/model/rb_link3.STL; visual mesh filename=package://dog/model/rb_link3.STL
- link rb_link4: mass 0.432627455975136 -> 0.432627455975141; geometry collision mesh filename=package://dog/model/rb_link4.STL; visual mesh filename=package://dog/model/rb_link4.STL
- link rf_link1: mass 0.305258520879219 -> 0.305258520879218; geometry collision mesh filename=package://dog/model/rf_link1.STL; visual mesh filename=package://dog/model/rf_link1.STL
- link rf_link2: mass 0.682338731946652 -> 0.682338731946651; geometry collision mesh filename=package://dog/model/rf_link2.STL; visual mesh filename=package://dog/model/rf_link2.STL
- link rf_link3: geometry collision mesh filename=package://dog/model/rf_link3.STL; visual mesh filename=package://dog/model/rf_link3.STL
- link rf_link4: mass 0.43262756992202 -> 0.432627569922017; geometry collision mesh filename=package://dog/model/rf_link4.STL; visual mesh filename=package://dog/model/rf_link4.STL
Joints:
- joint lb_joint1: axis 0 0 -1 -> 0 0 1; limit lower=0 upper=0 effort=0 velocity=0 -> lower=-3 upper=3 effort=20 velocity=16
- joint lb_joint2: axis 0 0 -1 -> 0 0 1; limit lower=0 upper=0 effort=0 velocity=0 -> lower=-3 upper=3 effort=20 velocity=16; origin xyz=-0.00047387 -0.029283 0.059987 rpy=-1.5708 0 3.1254 -> xyz=-0.00047387 -0.029283 0.059987 rpy=1.5708 -0.67742 -0.016174
- joint lb_joint3: axis 0 0 -1 -> 0 0 1; limit lower=0 upper=0 effort=0 velocity=0 -> lower=-3 upper=3 effort=20 velocity=16; origin xyz=-0.17921 -0.14417 0.0935 rpy=0 0 2.6627 -> xyz=0.23001 1.0811E-05 0.0935 rpy=0 0 -1.1563
- joint lb_joint4: axis 0 0 -1 -> 0 0 1
- joint lf_joint1: axis 0 0 -1 -> 0 0 1; limit lower=0 upper=0 effort=0 velocity=0 -> lower=-3 upper=3 effort=20 velocity=16
- joint lf_joint2: axis 0 0 -1 -> 0 0 1; limit lower=0 upper=0 effort=0 velocity=0 -> lower=-3 upper=3 effort=20 velocity=16; origin xyz=0 0.029313 0.060013 rpy=1.5708 0 3.1416 -> xyz=0 0.029313 0.060013 rpy=-1.5708 0.87219 0
- joint lf_joint3: axis 0 0 -1 -> 0 0 1; limit lower=0 upper=0 effort=0 velocity=0 -> lower=-3 upper=3 effort=20 velocity=16; origin xyz=-0.14792 -0.17613 0.0935 rpy=0 0 -1.5708 -> xyz=0.23001 0 0.0935 rpy=0 0 -1.74
- joint lf_joint4: axis 0 0 -1 -> 0 0 1; origin xyz=-0.17165 -0.14547 0.028 rpy=0 0 0 -> xyz=0.225 0 0.028 rpy=0 0 2.4386
- joint rb_joint1: axis 0 0 -1 -> 0 0 1; limit lower=0 upper=0 effort=0 velocity=0 -> lower=-3 upper=3 effort=20 velocity=16
- joint rb_joint2: axis 0 0 -1 -> 0 0 1; limit lower=0 upper=0 effort=0 velocity=0 -> lower=-3 upper=3 effort=20 velocity=16; origin xyz=-0.001301 0.029271 0.06 rpy=-1.5708 0 0.044416 -> xyz=-0.001301 0.029271 0.06 rpy=-1.5708 -0.56823 0.044416
- joint rb_joint3: axis 0 0 -1 -> 0 0 1; limit lower=0 upper=0 effort=0 velocity=0 -> lower=-3 upper=3 effort=20 velocity=16; origin xyz=0.19386 -0.12377 0.0935 rpy=0 0 0.53404 -> xyz=0.23 0 0.0935 rpy=0 0 1.1023
- joint rb_joint4: axis 0 0 -1 -> 0 0 1
- joint rf_joint1: axis 0 0 -1 -> 0 0 1; limit lower=0 upper=0 effort=0 velocity=0 -> lower=-3 upper=3 effort=20 velocity=16
- joint rf_joint2: axis 0 0 -1 -> 0 0 1; limit lower=0 upper=0 effort=0 velocity=0 -> lower=-3 upper=3 effort=20 velocity=16; origin xyz=0 -0.029287 0.059987 rpy=1.5708 -1.5708 0 -> xyz=0 -0.029287 0.059987 rpy=1.5708 0.63231 0
- joint rf_joint3: axis 0 0 -1 -> 0 0 1; limit lower=0 upper=0 effort=0 velocity=0 -> lower=-3 upper=3 effort=20 velocity=16; origin xyz=-0.13592 -0.18553 0.0935 rpy=0 0 -0.80414 -> xyz=0.22999 1.0192E-05 0.0935 rpy=0 0 1.399
- joint rf_joint4: axis 0 0 -1 -> 0 0 1
