Commit message: 6

File: src/dog/arm/arm.urdf (robot description, URDF)
Before this commit: robot arm, 5 links, 4 joints
Joints:
- joint joint1: limit lower=0 upper=0 effort=0 velocity=0 -> lower=-1 upper=1 effort=0 velocity=0
- joint joint2: axis 0 1 0 -> 0 0 1; limit lower=0 upper=0 effort=0 velocity=0 -> lower=-1 upper=1 effort=0 velocity=0; parent base_link -> link1
- joint joint3: axis 0 1 0 -> 0 0 1; limit lower=0 upper=0 effort=0 velocity=0 -> lower=-1 upper=1 effort=0 velocity=0; parent base_link -> link2
- joint joint4: axis 0 1 0 -> 0 0 1; limit lower=0 upper=0 effort=0 velocity=0 -> lower=-1 upper=1 effort=0 velocity=0; parent base_link -> link3
